Commit message: fix: add task 3

File: ex03/my_robot/urdf/robot.gazebo.xacro (robot description, xacro)
@@ -27,6 +27,6 @@
             <right_joint>right_wheel_joint</right_joint>
             <child_frame_id>robot/base_link</child_frame_id>
-            <wheel_separation>0.291</wheel_separation>
-            <wheel_radius>0.033</wheel_radius>
+            <wheel_separation>0.31</wheel_separation>
+            <wheel_radius>0.05</wheel_radius>
             <odom_publish_frequency>10</odom_publish_frequency>
         </plugin>

File: ex03/my_robot/urdf/robot.urdf.xacro (robot description, xacro)
@@ -4,12 +4,12 @@
     <!--xacro:include filename="$(find robot_description)/urdf/lidar.urdf.xacro" /-->
     <!--xacro:include filename="$(find robot_description)/urdf/depth.urdf.xacro" /-->
-    <xacro:property name="chassis_length" value="0.335"/>
-    <xacro:property name="chassis_width" value="0.265"/>
-    <xacro:property name="chassis_height" value="0.138"/>
+    <xacro:property name="chassis_length" value="0.15"/>
+    <xacro:property name="chassis_width" value="0.13"/>
+    <xacro:property name="chassis_height" value="0.07"/>
     <xacro:property name="wheel_radius" value="0.033"/>
     <xacro:property name="wheel_thickness" value="0.026"/>
     <xacro:property name="wheel_mass" value="0.05"/>
-    <xacro:property name="wheel_offset_x" value="0.226"/>
-    <xacro:property name="wheel_offset_y" value="0.1485"/>
+    <xacro:property name="wheel_offset_x" value="0.1"/>
+    <xacro:property name="wheel_offset_y" value="0.07"/>
     <xacro:property name="wheel_offset_z" value="0.01"/>
     <xacro:property name="caster_wheel_radius" value="0.01"/>
